Commit message: updating IMU position

File: src/sim/description/imu.xacro (robot description, xacro)
@@ -4,5 +4,5 @@
         <parent link="chassis"/>
         <child link="imu_link"/>
-        <origin xyz="-0.1 0 0.1" rpy="0 0 0"/>
+        <origin xyz="0.04 0 0.15" rpy="0 0 0"/>
     </joint>
     <link name="imu_link">
